File: pwrconv.kicad_sch (KiCad schematic)
At the start: 31 parts, among them J1 Power In, J2 Power Out, U1 TPS5430DDA, U2 TPS5430DDA, U3 TPS5430DDA

Commit message: Add files via upload
Parts:
- removed C1: 4.7 μF, Capacitor_SMD:C_0603_1608Metric, symbol Device:C
- removed C11: 100 μF, Capacitor_SMD:C_0603_1608Metric, symbol Device:C
- removed C12: 1500 pF, Capacitor_SMD:C_0603_1608Metric, symbol Device:C
- removed C6: 0.01 μF, Capacitor_SMD:C_0603_1608Metric, symbol Device:C
- removed C7: 150 pF, Capacitor_SMD:C_0603_1608Metric, symbol Device:C
- removed C8: 0.1 μF, Capacitor_SMD:C_0603_1608Metric, symbol Device:C
- removed D3: D_Schottky, Diode_SMD:D_0603_1608Metric, symbol Device:D_Schottky
- removed J2: Power Out, Connector_PinHeader_2.54mm:PinHeader_1x04_P2.54mm_Vertical, symbol Connector:Conn_01x04_Pin
- removed L3: 15 μH, Inductor_SMD:L_0603_1608Metric, symbol Device:L_Iron
- removed R1: 549 Ω, Resistor_SMD:R_0603_1608Metric, symbol Device:R
- removed R4: 5.9 kΩ, Resistor_SMD:R_0603_1608Metric, symbol Device:R
- removed R7: 10 kΩ, Resistor_SMD:R_0603_1608Metric, symbol Device:R
- removed U3: TPS5430DDA, Package_SO:TI_SO-PowerPAD-8_ThermalVias, symbol Regulator_Switching:TPS5430DDA
- added J2: Power Out, Connector_PinHeader_2.54mm:PinHeader_1x03_P2.54mm_Vertical, symbol Connector:Conn_01x03_Pin
- added L3, L5: 10uH, Inductor_SMD:L_Changjiang_FXL0630, symbol Device:L
- C1: renamed from C3; footprint Capacitor_SMD:C_0603_1608Metric -> Capacitor_SMD:C_0805_2012Metric; LCSC (none) -> C1779
- C2: value 10u -> 4.7uF; footprint Capacitor_SMD:C_0603_1608Metric -> Capacitor_SMD:C_0805_2012Metric; LCSC (none) -> C1779
- C3: renamed from C4; LCSC (none) -> C1589
- C4: renamed from C5; LCSC (none) -> C1589
- C5: renamed from C9; value 220uF -> 100uF; footprint Capacitor_SMD:C_0603_1608Metric -> Capacitor_SMD:C_Elec_6.3x7.7; LCSC (none) -> C2836437
- C6: renamed from C10; footprint Capacitor_SMD:C_0603_1608Metric -> Capacitor_SMD:C_0805_2012Metric; LCSC (none) -> C45783
- D1, D2: footprint Diode_SMD:D_0603_1608Metric -> Diode_SMD:D_SOD-323; LCSC (none) -> C191023
- L1: value 10u -> 10uH; footprint (none) -> Inductor_SMD:L_Changjiang_FXL0630; LCSC (none) -> C167223
- L2: value >=26 uH -> 10uH; footprint Inductor_SMD:L_0603_1608Metric -> Inductor_SMD:L_Changjiang_FXL0630; LCSC (none) -> C167223
- L4: value 12u -> 10uH; footprint (none) -> Inductor_SMD:L_Changjiang_FXL0630; LCSC (none) -> C167223
- R1: renamed from R5; LCSC (none) -> C15401
- R2: renamed from R6; value 3.2K -> 3.3K; footprint Resistor_SMD:R_0603_1608Metric -> Resistor_SMD:R_1206_3216Metric; LCSC (none) -> C26041
- R3: renamed from R2; LCSC (none) -> C15401
- R4: renamed from R3; value 1.13k -> 1k; footprint Resistor_SMD:R_0603_1608Metric -> Resistor_SMD:R_1206_3216Metric; LCSC (none) -> C4410
- U1, U2: LCSC (none) -> C9864
Connections:
- net +12V: now also J2.1 (Pin_1), L5.2; no longer L4.2
- net +5V: now also J2.2 (Pin_2), L3.2; no longer L2.2
- net GND: now also J2.3 (Pin_3)
- net at C3.2, D1.1 (K), U1.8 (PH): now also L1.1; no longer L2.1
- net at L1.2: now also L3.1; no longer L4.1
- net at C4.2, D2.1 (K), U2.8 (PH): now also L2.1; no longer L1.1
- new net: L2.2, L4.1
- new net: L4.2, L5.1
- no-connect marks 3 -> 2
Other:
- moved on the sheet: C2, C3, C4, C5, C6, J1, R1, R2, R3, R4
