File: EPS PCB/EPS_PCB_Prototyping/Hysteresis_circ.kicad_sch (KiCad schematic)
At the start: 8 parts, among them U8 TLV3691IDPFR

Commit message: Prototyping Board Added
Parts:
- R23, R24, R26, R27: footprint Resistor_SMD:R_1206_3216Metric -> Resistor_THT:R_Axial_DIN0207_L6.3mm_D2.5mm_P7.62mm_Horizontal
Changed lines of the file:
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@@
 			)
 		)
-		(property "Footprint" "Resistor_SMD:R_1206_3216Metric"
+		(property "Footprint" "Resistor_THT:R_Axial_DIN0207_L6.3mm_D2.5mm_P7.62mm_Horizontal"
 			(at 106.2381 82.1059 90)
 			(effects
@@
 			)
 		)
-		(property "Footprint" "Resistor_SMD:R_1206_3216Metric"
+		(property "Footprint" "Resistor_THT:R_Axial_DIN0207_L6.3mm_D2.5mm_P7.62mm_Horizontal"
 			(at 94.4323 96.5025 90)
 			(effects
@@
 			)
 		)
-		(property "Footprint" "Resistor_SMD:R_1206_3216Metric"
+		(property "Footprint" "Resistor_THT:R_Axial_DIN0207_L6.3mm_D2.5mm_P7.62mm_Horizontal"
 			(at 121.3764 82.1059 90)
 			(effects
@@
 			)
 		)
-		(property "Footprint" "Resistor_SMD:R_1206_3216Metric"
+		(property "Footprint" "Resistor_THT:R_Axial_DIN0207_L6.3mm_D2.5mm_P7.62mm_Horizontal"
 			(at 94.4323 40.6225 90)
 			(effects

Commit message: EPS PCB Prototype For order
yea
Parts:
- added J11, J12: Conn_01x02_Pin, Connector_PinSocket_2.54mm:PinSocket_1x02_P2.54mm_Vertical, symbol Connector:Conn_01x02_Pin
Connections:
- net 5V_conv_out: now also J11.2 (Pin_2); no longer R26.1, U8.6 (VCC)
- new net: J11.1 (Pin_1), J12.2 (Pin_2), R26.1, U8.6 (VCC)
- new net +5Vin2: J12.1 (Pin_1)
