File: EPS PCB/EPS_PCB_Prototyping/curr_meas.kicad_sch (KiCad schematic)
At the start: 30 parts, among them Q1 DMN3016LFDE-7, Q2 DMN3016LFDE-7, Q3 DMN3016LFDE-7, U5 INA3221, U6 STEF033APUR, U7 STEF512PUR

Commit message: Prototype board v1 finished
Connections:
- net IN+4 is gone; now on net 3V3_to_fuse: U5.1 (IN-3)
- net 3V3_conv_out: now also C13.1, C24.1, R11.1, R12.1, R13.1, R14.1, R15.1, R16.1, U5.16 (VPU)
- net 3V3_out: no longer C13.1, C24.1, R11.1, R12.1, R13.1, R14.1, R15.1, R16.1, U5.16 (VPU)
Changed lines of the file:
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@@
 		)
 	)
-	(label "IN+4"
+	(label "IN-3"
 		(at 109.22 59.69 0)
 		(effects
@@
 		)
 	)
-	(global_label "3V3_out"
+	(global_label "3V3_conv_out"
 		(shape input)
 		(at 201.93 36.83 90)
@@
 		)
 		(property "Intersheetrefs" "${INTERSHEET_REFS}"
-			(at 201.93 26.3459 90)
+			(at 201.93 21.0241 90)
 			(effects
 				(font
@@
 		)
 	)
-	(global_label "3V3_out"
+	(global_label "3V3_conv_out"
 		(shape input)
 		(at 129.54 22.86 90)
@@
 		)
 		(property "Intersheetrefs" "${INTERSHEET_REFS}"
-			(at 129.54 12.3759 90)
+			(at 129.54 7.0541 90)
 			(effects
 				(font
@@
 		)
 	)
-	(global_label "3V3_out"
+	(global_label "3V3_conv_out"
 		(shape input)
 		(at 124.46 22.86 90)
@@
 		)
 		(property "Intersheetrefs" "${INTERSHEET_REFS}"
-			(at 124.46 12.3759 90)
+			(at 124.46 7.0541 90)
 			(effects
 				(font
@@
 		)
 	)
-	(global_label "3V3_out"
+	(global_label "3V3_conv_out"
 		(shape input)
 		(at 109.8299 25.2831 90)
@@
 		)
 		(property "Intersheetrefs" "${INTERSHEET_REFS}"
-			(at 109.8299 14.799 90)
+			(at 109.8299 9.4772 90)
 			(effects
 				(font
@@
 		(lib_id "Device:C")
 		(at 100.33 86.36 0)
+		(mirror y)
 		(unit 1)
 		(exclude_from_sim no)
@@
 		(dnp no)
 		(property "Reference" "C14"
-			(at 104.14 85.0899 0)
+			(at 96.52 85.0899 0)
 			(effects
 				(font
@@
 		)
 		(property "Value" "10u"
-			(at 104.14 87.6299 0)
+			(at 96.52 87.6299 0)
 			(effects
 				(font
@@
 		)
 		(property "Footprint" "Capacitor_SMD:C_0603_1608Metric"
-			(at 101.2952 90.17 0)
-			(effects
-				(font
+			(at 99.3648 90.17 0)
+			(effects
+				(font

Commit message: EPS PCB Prototype For order
yea
Parts:
- added J10, J8, J9: Conn_01x02_Pin, Connector_PinSocket_2.54mm:PinSocket_1x02_P2.54mm_Vertical, symbol Connector:Conn_01x02_Pin
Connections:
- net 12V_to_fuse: now also J9.1 (Pin_1); no longer R9.2, U5.14 (IN-2)
- net 3V3_to_fuse: now also J10.1 (Pin_1); no longer R10.2, U5.1 (IN-3)
- net 5V_to_fuse: now also J8.1 (Pin_1); no longer R8.2, U5.11 (IN-1)
- new net IN-1: J8.2 (Pin_2), R8.2, U5.11 (IN-1)
- new net IN-2: J9.2 (Pin_2), R9.2, U5.14 (IN-2)
- new net IN-3: J10.2 (Pin_2), R10.2, U5.1 (IN-3)
