File: EPS PCB/EPS_PCB_Prototyping/pwrconv.kicad_sch (KiCad schematic)
At the start: 27 parts, among them U1 TPS5430DDA, U2 TPS5430DDA, U3 TPS5430DDA

Commit message: Prototype board v1 finished
Parts:
- C7: footprint Capacitor_SMD:C_Elec_6.3x7.7 -> Capacitor_SMD:C_0805_2012Metric
Connections:
- net 12V_out renamed 12V_conv_out
- net 3V3_out renamed 3V3_conv_out
- net 5V_out renamed 5V_conv_out
Changed lines of the file:
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@@
 		)
 	)
-	(global_label "3V3_out"
+	(global_label "3V3_conv_out"
 		(shape input)
 		(at 152.4 120.65 0)
@@
 		)
 		(property "Intersheetrefs" "${INTERSHEET_REFS}"
-			(at 162.8841 120.65 0)
+			(at 168.2059 120.65 0)
 			(effects
 				(font
@@
 		)
 	)
-	(global_label "5V_out"
+	(global_label "5V_conv_out"
 		(shape input)
 		(at 142.24 24.13 0)
@@
 		)
 		(property "Intersheetrefs" "${INTERSHEET_REFS}"
-			(at 151.5146 24.13 0)
-			(effects
-				(font
-					(size 1.27 1.27)
-				)
-				(justify left)
-				(hide yes)
-			)
-		)
-	)
-	(global_label "12V_out"
+			(at 156.8364 24.13 0)
+			(effects
+				(font
+					(size 1.27 1.27)
+				)
+				(justify left)
+				(hide yes)
+			)
+		)
+	)
+	(global_label "12V_conv_out"
 		(shape input)
 		(at 152.4 67.31 0)
@@
 		)
 		(property "Intersheetrefs" "${INTERSHEET_REFS}"
-			(at 162.8841 67.31 0)
+			(at 168.2059 67.31 0)
 			(effects
 				(font
@@
 			)
 		)
-		(property "Footprint" "Capacitor_SMD:C_Elec_6.3x7.7"
+		(property "Footprint" "Capacitor_SMD:C_0805_2012Metric"
 			(at 127.9652 46.99 0)
 			(effects

Commit message: EPS PCB Prototype For order
yea
Parts:
- added J3, J4, J5: Conn_01x02_Pin, Connector_PinSocket_2.54mm:PinSocket_1x02_P2.54mm_Vertical, symbol Connector:Conn_01x02_Pin
Connections:
- net 12V_conv_out: now also J4.2 (Pin_2); no longer C8.2, L6.2, R3.1
- net 3V3_conv_out: now also J5.2 (Pin_2); no longer C9.2, L3.2, R5.1
- net 5V_conv_out: now also J3.2 (Pin_2); no longer C7.1, L4.2, R1.1
- new net: C7.1, J3.1 (Pin_1), L4.2, R1.1
- new net: C8.2, J4.1 (Pin_1), L6.2, R3.1
- new net: C9.2, J5.1 (Pin_1), L3.2, R5.1
