File: EPS PCB/EPS_PCB_Prototyping/EPS_PCB_Prototyping.kicad_pcb (KiCad board)
At the start: 2 copper layers, 95.9 x 90.2 mm, 82 parts, among them J1 Conn_02x32_Row_Letter_First, J2 Conn_02x20_Row_Letter_First, J3 Power In, J4 Power Out, Q1 DMN3016LFDE-7, Q2 DMN3016LFDE-7, Q3 DMN3016LFDE-7, U1 TPS5430DDA, U2 TPS5430DDA, U3 TPS5430DDA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

Commit message: Prototype board v1 finished
Parts:
- removed H5, H6, H7, H8: MountingHole, MountingHole:MountingHole_2mm
- removed J3: Power In, Connector_PinHeader_2.54mm:PinHeader_1x02_P2.54mm_Vertical
- removed J4: Power Out, Connector_PinHeader_2.54mm:PinHeader_1x02_P2.54mm_Vertical
- C7: footprint Capacitor_SMD:C_Elec_6.3x7.7 -> Capacitor_SMD:C_0805_2012Metric
- moved R24 188.5 mm to (213.2, 58.2), turned to 90 degrees
- moved R27 183.8 mm to (208.4, 67.3), turned to 90 degrees
- moved R23 178.3 mm to (204.2, 58.9), turned to -90 degrees
- moved R22 175.8 mm to (215.9, 69.8), turned to 90 degrees
- moved U8 174.0 mm to (212.2, 69.8), turned to 90 degrees
- moved R21 173.1 mm to (215.9, 74.0), turned to 90 degrees
- moved R26 173.0 mm to (199.4, 69.4), turned to 90 degrees
- moved R20 170.6 mm to (215.9, 78.0), turned to 90 degrees
- moved C3 163.2 mm to (213.5, 128.8), turned to -90 degrees
- moved U3 162.6 mm to (208.3, 128.9)
- moved C2 160.1 mm to (214.2, 108.3), turned to -90 degrees
- moved L3 159.1 mm to (199.8, 120.9), turned to 180 degrees
- moved L1 158.9 mm to (206.4, 75.8), turned to 180 degrees
- moved L2 158.6 mm to (203.5, 97.6), turned to 180 degrees
- moved U2 158.2 mm to (208.8, 108.3)
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Connections:
- C12 pad 1: +3.3V -> 5V_conv_out
- C13 pad 1: 3V3_out -> 3V3_conv_out
- C24 pad 1: 3V3_out -> 3V3_conv_out
- C7 pad 1: 5V_out -> 5V_conv_out
- C8 pad 2: 12V_out -> 12V_conv_out
- C9 pad 2: 3V3_out -> 3V3_conv_out
- J1 pad a14: unconnected-(J1-Pin_a14-Pada14) -> A0
- J1 pad a15: unconnected-(J1-Pin_a15-Pada15) -> CM_SCL
- J1 pad a16: unconnected-(J1-Pin_a16-Pada16) -> CM_SDA
- J1 pad a17: unconnected-(J1-Pin_a17-Pada17) -> WARNING
- J1 pad a18: unconnected-(J1-Pin_a18-Pada18) -> CRITICAL
- J1 pad a19: unconnected-(J1-Pin_a19-Pada19) -> PV
- J1 pad a3: unconnected-(J1-Pin_a3-Pada3) -> 5V_en
- J1 pad a30: unconnected-(J1-Pin_a30-Pada30) -> GPIO
- J1 pad a5: unconnected-(J1-Pin_a5-Pada5) -> 3V3_en
- J1 pad a9: unconnected-(J1-Pin_a9-Pada9) -> 12V_en
- J1 pad b15: unconnected-(J1-Pin_b15-Padb15) -> 3V3_conv_out
- J1 pad b16: unconnected-(J1-Pin_b16-Padb16) -> 5V_conv_out
- J1 pad b17: unconnected-(J1-Pin_b17-Padb17) -> 12V_conv_out
- J1 pad b2: RESET -> unconnected-(J1-Pin_b2-Padb2)
- J1 pad b29: unconnected-(J1-Pin_b29-Padb29) -> HYST_OUT
- J1 pad b3: +5V -> 5V_out
- J1 pad b30: unconnected-(J1-Pin_b30-Padb30) -> RESET
- J1 pad b5: +3.3V -> 3V3_out
- J1 pad b6: unconnected-(J1-Pin_b6-Padb6) -> V_Batt
- J1 pad b8: unconnected-(J1-Pin_b8-Padb8) -> V_Batt
- J1 pad b9: +12V -> 12V_out
- L3 pad 2: 3V3_out -> 3V3_conv_out
- L4 pad 2: 5V_out -> 5V_conv_out
- L6 pad 2: 12V_out -> 12V_conv_out
- R1 pad 1: 5V_out -> 5V_conv_out
- R11 pad 1: 3V3_out -> 3V3_conv_out
- R12 pad 1: 3V3_out -> 3V3_conv_out
- R13 pad 1: 3V3_out -> 3V3_conv_out
- R14 pad 1: 3V3_out -> 3V3_conv_out
- R15 pad 1: 3V3_out -> 3V3_conv_out
- R16 pad 1: 3V3_out -> 3V3_conv_out
- R3 pad 1: 12V_out -> 12V_conv_out
- R5 pad 1: 3V3_out -> 3V3_conv_out
- R7 pad 1: +3.3V -> 5V_conv_out
- U4 pad 3: +3.3V -> 5V_conv_out
- U4 pad 5: +3.3V -> 5V_conv_out
- U5 pad 1: /Curr_meas/IN+4 -> /Curr_meas/3V3_to_fuse
- U5 pad 16: 3V3_out -> 3V3_conv_out
Routing:
- net 3V3_conv_out: track 0.00 -> 132.0 mm, vias 0 -> 9
- net 5V_conv_out: track 0.00 -> 130.0 mm
- net 12V_conv_out: track 0.00 -> 96.3 mm, vias 0 -> 4
- net GND: track 0.00 -> 78.6 mm, vias 0 -> 16
- net /Curr_meas/12V_to_fet: track 0.00 -> 75.2 mm, vias 0 -> 2
- net WARNING: track 0.00 -> 73.4 mm, vias 0 -> 3
- net CRITICAL: track 0.00 -> 69.0 mm, vias 0 -> 3
- net PV: track 0.00 -> 68.6 mm, vias 0 -> 3
- net A0: track 0.00 -> 66.7 mm, vias 0 -> 2
- net CM_SCL: track 0.00 -> 66.6 mm, vias 0 -> 2
- net /Curr_meas/5V_to_fet: track 0.00 -> 61.4 mm, vias 0 -> 2
- net CM_SDA: track 0.00 -> 58.4 mm, vias 0 -> 2
- net /Curr_meas/3V3_to_fet: track 0.00 -> 56.7 mm, vias 0 -> 2
- net RESET: track 0.00 -> 52.3 mm, vias 0 -> 1
- net GPIO: track 0.00 -> 52.2 mm, vias 0 -> 1
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- added copper zone on B.Cu, net V_Batt
Other:
- board text removed: "A1"
- board text removed: "A30"
- board text removed: "B"
- board text removed: "C"
- board text removed: "D1"
- board text removed: "D30"

Commit message: EPS PCB Prototype For order
yea
Parts:
- added J10: Conn_01x02_Pin, Connector_PinSocket_2.54mm:PinSocket_1x02_P2.54mm_Vertical, F.Cu at (172.4, 122.7)
- added J11: Conn_01x02_Pin, Connector_PinSocket_2.54mm:PinSocket_1x02_P2.54mm_Vertical, F.Cu at (205.8, 70.4)
- added J12: Conn_01x02_Pin, Connector_PinSocket_2.54mm:PinSocket_1x02_P2.54mm_Vertical, F.Cu at (216.3, 64.2)
- added J3: Conn_01x02_Pin, Connector_PinSocket_2.54mm:PinSocket_1x02_P2.54mm_Vertical, F.Cu at (198.0, 81.3)
- added J4: Conn_01x02_Pin, Connector_PinSocket_2.54mm:PinSocket_1x02_P2.54mm_Vertical, F.Cu at (203.2, 107.9)
- added J5: Conn_01x02_Pin, Connector_PinSocket_2.54mm:PinSocket_1x02_P2.54mm_Vertical, F.Cu at (197.2, 115.5)
- added J6: Conn_01x02_Pin, Connector_PinSocket_2.54mm:PinSocket_1x02_P2.54mm_Vertical, F.Cu at (190.7, 62.4)
- added J7: Conn_01x02_Pin, Connector_PinSocket_2.54mm:PinSocket_1x02_P2.54mm_Vertical, F.Cu at (185.9, 59.5)
- added J8: Conn_01x02_Pin, Connector_PinSocket_2.54mm:PinSocket_1x02_P2.54mm_Vertical, F.Cu at (183.9, 99.0)
- added J9: Conn_01x02_Pin, Connector_PinSocket_2.54mm:PinSocket_1x02_P2.54mm_Vertical, F.Cu at (172.9, 106.3)
Connections:
- C12 pad 1: 5V_conv_out -> /watchdog_timer/conn
- C7 pad 1: 5V_conv_out -> Net-(J3-Pin_1)
- C8 pad 2: 12V_conv_out -> Net-(J4-Pin_1)
- C9 pad 2: 3V3_conv_out -> Net-(J5-Pin_1)
- J2 pad d16: +5V -> unconnected-(J2-Pin_d16-Padd16)
- L3 pad 2: 3V3_conv_out -> Net-(J5-Pin_1)
- L4 pad 2: 5V_conv_out -> Net-(J3-Pin_1)
- L6 pad 2: 12V_conv_out -> Net-(J4-Pin_1)
- R1 pad 1: 5V_conv_out -> Net-(J3-Pin_1)
- R10 pad 2: /Curr_meas/3V3_to_fuse -> /Curr_meas/IN-3
- R26 pad 1: 5V_conv_out -> Net-(J11-Pin_1)
- R3 pad 1: 12V_conv_out -> Net-(J4-Pin_1)
- R5 pad 1: 3V3_conv_out -> Net-(J5-Pin_1)
- R7 pad 1: 5V_conv_out -> /watchdog_timer/conn
- R8 pad 2: /Curr_meas/5V_to_fuse -> /Curr_meas/IN-1
- R9 pad 2: /Curr_meas/12V_to_fuse -> /Curr_meas/IN-2
- U4 pad 3: 5V_conv_out -> Net-(U4-EN)
- U4 pad 5: 5V_conv_out -> Net-(U4-EN)
- U5 pad 1: /Curr_meas/3V3_to_fuse -> /Curr_meas/IN-3
- U5 pad 11: /Curr_meas/5V_to_fuse -> /Curr_meas/IN-1
- U5 pad 14: /Curr_meas/12V_to_fuse -> /Curr_meas/IN-2
- U8 pad 6: 5V_conv_out -> Net-(J11-Pin_1)
Routing:
- net Net-(J11-Pin_1): track 0.00 -> 25.9 mm
- net 5V_conv_out: track 130.0 -> 112.0 mm, vias 0 -> 2
- net 3V3_conv_out: track 132.0 -> 114.5 mm
- net Net-(J5-Pin_1): track 0.00 -> 14.8 mm
- net /Curr_meas/5V_to_fuse: track 35.2 -> 20.9 mm, vias 2 -> 1
- net Net-(J4-Pin_1): track 0.00 -> 13.5 mm
- net /watchdog_timer/conn: track 0.00 -> 12.8 mm
- net /Curr_meas/12V_to_fuse: track 34.5 -> 21.7 mm, vias 2 -> 1
- net /Curr_meas/IN-1: track 0.00 -> 11.7 mm
- net /Curr_meas/IN-2: track 0.00 -> 11.7 mm
- net /Curr_meas/IN-3: track 0.00 -> 10.8 mm
- net Net-(J3-Pin_1): track 0.00 -> 9.41 mm
- net Net-(U4-EN): track 0.00 -> 7.47 mm, vias 0 -> 2
- net /Curr_meas/3V3_to_fuse: track 18.9 -> 12.4 mm
- net A0: track 66.7 -> 71.5 mm
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Other:
- board text added: "5V in"
- board text added: "5v in"
- board text added: "B"
