File: PCI-104-Temp/PCI-104-Temp/PCI-104-Temp.kicad_pcb (KiCad board)
At the start: 2 copper layers, 95.9 x 90.2 mm, 6 parts, among them J1 Conn_02x32_Row_Letter_First, J2 Conn_02x20_Row_Letter_First

Commit message: PC104 Template Updated
Parts:
- removed J1: Conn_02x32_Row_Letter_First, Connector_PinHeader_2.54mm:PinHeader_2x32_P2.54mm_Vertical
- removed J2: Conn_02x20_Row_Letter_First, Connector_PinHeader_2.54mm:PinHeader_2x20_P2.54mm_Vertical
- added J3: Conn_02x26_Row_Letter_First, Connector_PinSocket_2.54mm:PinSocket_2x26_P2.54mm_Vertical, F.Cu at (221.9, 62.1)
- added J4: Conn_02x26_Row_Letter_First, Connector_PinSocket_2.54mm:PinSocket_2x26_P2.54mm_Vertical, F.Cu at (227.0, 62.1)
- moved H2 3.81 mm to (227.0, 57.0)
- moved H3 3.81 mm to (141.3, 133.2)
- moved H4 2.54 mm to (227.0, 130.7)
- moved H1 2.54 mm to (141.3, 53.2)
