File: PCI-104-Temp/PCI-104-Temp/PCI-104.kicad_sch (KiCad schematic)
At the start: 6 parts, among them J1 Conn_02x32_Row_Letter_First, J2 Conn_02x20_Row_Letter_First

Commit message: PC104 Template Updated
Parts:
- removed J1: Conn_02x32_Row_Letter_First, Connector_PinSocket_2.54mm:PinSocket_2x32_P2.54mm_Vertical, symbol Connector_Generic:Conn_02x32_Row_Letter_First
- removed J2: Conn_02x20_Row_Letter_First, Connector_PinSocket_2.54mm:PinSocket_2x20_P2.54mm_Vertical, symbol Connector_Generic:Conn_02x20_Row_Letter_First
- added J3, J4: Conn_02x26_Row_Letter_First, Connector_PinSocket_2.54mm:PinSocket_2x26_P2.54mm_Vertical, symbol Connector_Generic:Conn_02x26_Row_Letter_First
Connections:
- net GND: now also J3.a26 (Pin_a26), J3.b26 (Pin_b26), J4.a26 (Pin_a26)
