File: EPS PCB/EPS_PCB_PrototypingV2/curr_meas.kicad_sch (KiCad schematic)
At the start: 33 parts, among them J10 Conn_01x02_Pin, J8 Conn_01x02_Pin, J9 Conn_01x02_Pin, Q1 DMN3016LFDE-7, Q2 DMN3016LFDE-7, Q3 DMN3016LFDE-7, U5 INA3221, U6 STEF033APUR, U7 STEF512PUR

Commit message: PC104 Template Updates
Parts:
- removed J10, J8, J9: Conn_01x02_Pin, Connector_PinSocket_2.54mm:PinSocket_1x02_P2.54mm_Vertical, symbol Connector:Conn_01x02_Pin
- removed Q1, Q2, Q3: DMN3016LFDE-7, Footprints:TRANS_DMN3016LFDE-7, symbol DMN3016LFDE-7:DMN3016LFDE-7
- added Q1, Q2, Q5: DMG6968U, Package_TO_SOT_SMD:SOT-23-3, symbol Simulation_SPICE:PMOS
- added Q3, Q4, Q6: 2N7002, Package_TO_SOT_SMD:SOT-23-3, symbol Simulation_SPICE:NMOS
- added R19, R21, R22: 10k, Resistor_SMD:R_1206_3216Metric, symbol Device:R
- U7: footprint Footprints:STEF512 -> Footprints:QFN10_2X3_STM-L
- renumbered C17 to C15, C15 to C16, C22 to C17, C14 to C19, C24 to C20, C23 to C21, C13 to C22, C21 to C23, C20 to C24, C19 to C25, C16 to C26, R9 to R10, R10 to R11, R17 to R12, R19 to R13, R13 to R14, R14 to R15, R15 to R16, R16 to R17, R12 to R18, R11 to R20, R18 to R8, R8 to R9, U5 to U8
Connections:
- net 12V_to_fuse is gone; now on net 12V_conv_out: C26.1, U7.10 (VIN_12)
- net 3V3_to_fuse is gone; now on net 3V3_conv_out: C19.1, U6.11 (EPAD)
- net 5V_to_fuse is gone; now on net 5V_conv_out: C16.1, U7.4 (VIN_5)
- net A0 is gone; now on net CM_SCL: U8.5 (A0)
- net IN-1 is gone; now on net 5V_to_fet: R9.2, U8.11 (IN-1)
- net IN-2 is gone; now on net 12V_to_fet: R10.2, U8.14 (IN-2)
- net IN-3 is gone; now on net 3V3_to_fet: R11.2, U8.1 (IN-3)
- net 12V_conv_out: no longer R10.1, U8.15 (IN+2)
- net 12V_en: now also Q4.2 (G)
- net 12V_out: now also Q2.1 (D)
- net 12V_to_fet: now also Q2.3 (S); no longer C25.1, U7.9 (VOUT_12)
- net 3V3_conv_out: no longer C20.1, C22.1, R11.1, R14.1, R15.1, R16.1, R17.1, R18.1, R20.1, U8.16 (VPU), U8.2 (IN+3)
- net 3V3_en: now also Q6.2 (G)
- net 3V3_out: now also C20.1, C22.1, R14.1, R15.1, R16.1, R17.1, R18.1, R20.1, U8.16 (VPU), Q5.1 (D)
- net 3V3_to_fet: now also Q5.3 (S); no longer C15.1, U6.1 (SOURCE), U6.2 (SOURCE), U6.3 (SOURCE), U6.4 (SOURCE), U6.5 (SOURCE)
- net 5V_conv_out: no longer R9.1, U8.12 (IN+1)
- net 5V_en: now also Q3.2 (G)
- net 5V_out: now also Q1.1 (D)
- net 5V_to_fet: now also Q1.3 (S); no longer C18.1, U7.5 (VOUT_5)
- net GND: now also Q3.3 (S), Q4.3 (S), Q6.3 (S)
- new net: Q5.2 (G), Q6.1 (D), R22.2
- new net: Q2.2 (G), Q4.1 (D), R21.2
- new net: Q1.2 (G), Q3.1 (D), R19.2
- new net 12V_to_cm: C25.1, R10.1, U7.9 (VOUT_12), U8.15 (IN+2)
- new net 3V3_to_cm: C15.1, R11.1, U6.1 (SOURCE), U6.2 (SOURCE), U6.3 (SOURCE), U6.4 (SOURCE), U6.5 (SOURCE), U8.2 (IN+3)
- new net 5V_HK: R19.1, R21.1, R22.1
- new net 5V_to_cm: C18.1, R9.1, U7.5 (VOUT_5), U8.12 (IN+1)
